Commit message: updated the urdf file

File: urdf/diffDriveTest.urdf.xacro (robot description, xacro)
@@ -1,6 +1,8 @@
 <?xml version="1.0"?>
 <robot name="roscontrol" xmlns:xacro="http://ros.org/wiki/xacro">
-    <xacro:property name="bodylen" value="0.6" />
-    <xacro:property name="width" value="0.2" />
+    <xacro:property name="WheelSep" value="0.26"/>
+    <xacro:property name="WheelRad" value="0.055"/>
+    <xacro:property name="WheelLen" value="0.1"/>
+    <xacro:property name="WheelPoss" value="0.15"/>
     <material name="blue">
         <color rgba="0 0 0.8 1"/>
@@ -21,5 +23,5 @@
         <visual>
             <geometry>
-                <cylinder radius="${width}" length="${bodylen}"/>
+                <box size="0.8 0.4 0.2"/>
             </geometry>
             <material name="blue"/>
@@ -27,8 +29,105 @@
         <collision>
             <geometry>
-                <cylinder radius="${width}" length="${bodylen}"/>
+                <box size="0.8 0.4 0.2"/>
             </geometry>
         </collision>
         <xacro:default_inertial mass="10"/>
     </link>
+    <!-- wheels -->
+    <xacro:macro name="wheels" params = "prefex reflect">
+        <!-- back wheels -->
+        <link name="${prefex}_back_wheel">
+            <visual>
+                <origin rpy="1.57075 0 0" xyz="0 0 0"/>
+                <geometry>
+                    <cylinder length="${WheelLen}" radius="${WheelRad}"/>
+                </geometry>
+                <material name="black"/>
+            </visual>
+            <collision>
+                <geometry>
+                    <cylinder length="${WheelLen}" radius="${WheelRad}"/>
+                </geometry>
+            </collision>
+            <xacro:default_inertial mass="1"/>
+        </link>
+        <joint name="${prefex}_back_wheel_joint" type="continuous">
+            <axis xyz="0 1 0" rpy="0 0 0" />
+            <parent link="base_link"/>
+            <child link="${prefex}_back_wheel"/>
+            <origin rpy="0 0 0" xyz="-${WheelPoss*2} ${reflect*WheelSep/2} -0.13"/>
+        </joint>
+        <link name="${prefex}_back_M_wheel">
+            <visual>
+                <origin rpy="1.57075 0 0" xyz="0 0 0"/>
+                <geometry>
+                    <cylinder length="${WheelLen}" radius="${WheelRad}"/>
+                </geometry>
+                <material name="black"/>
+            </visual>
+            <collision>
+                <geometry>
+                    <cylinder length="${WheelLen}" radius="${WheelRad}"/>
+                </geometry>
+            </collision>
+            <xacro:default_inertial mass="1"/>
+        </link>
+        <joint name="${prefex}_back_M_wheel_joint" type="continuous">
+            <axis xyz="0 1 0" rpy="0 0 0" />
+            <parent link="base_link"/>
+            <child link="${prefex}_back_M_wheel"/>
+            <origin rpy="0 0 0" xyz="-${WheelPoss} ${reflect*WheelSep/2} -0.13"/>
+        </joint>
+        <!-- front wheels -->
+        <link name="${prefex}_front_M_wheel">
+            <visual>
+                <origin rpy="1.57075 0 0" xyz="0 0 0"/>
+                <geometry>
+                    <cylinder length="${WheelLen}" radius="${WheelRad}"/>
+                </geometry>
+                <material name="black"/>
+            </visual>
+            <collision>
+                <geometry>
+                    <cylinder length="${WheelLen}" radius="${WheelRad}"/>
+                </geometry>
+            </collision>
+            <xacro:default_inertial mass="1"/>
+        </link>
+        <joint name="${prefex}_front_M_wheel_joint" type="continuous">
+            <axis xyz="0 1 0" rpy="0 0 0" />
+            <parent link="base_link"/>
+            <child link="${prefex}_front_M_wheel"/>
+            <origin rpy="0 0 0" xyz="${WheelPoss} ${reflect*WheelSep/2} -0.13"/>
+        </joint>
+        <link name="${prefex}_front_wheel">
+            <visual>
+                <origin rpy="1.57075 0 0" xyz="0 0 0"/>
+                <geometry>
+                    <cylinder length="${WheelLen}" radius="${WheelRad}"/>
+                </geometry>
+                <material name="black"/>
+            </visual>
+            <collision>
+                <geometry>
+                    <cylinder length="${WheelLen}" radius="${WheelRad}"/>
+                </geometry>
+            </collision>
+            <xacro:default_inertial mass="1"/>
+        </link>
+        <joint name="${prefex}_front_wheel_joint" type="continuous">
+            <axis xyz="0 1 0" rpy="0 0 0" />
+            <parent link="base_link"/>
+            <child link="${prefex}_front_wheel"/>
+            <origin rpy="0 0 0" xyz="${WheelPoss*2} ${reflect*WheelSep/2} -0.13"/>
+        </joint>
+    </xacro:macro>
+    <xacro:wheels prefex = "right" reflect = "-1"/>
+    <xacro:wheels prefex = "left" reflect = "1"/>
+    <!-- Gazebo plugin for ROS Control -->
+    <gazebo>
+        <plugin name="gazebo_ros_control" filename="libgazebo_ros_control.so">
+            <robotNamespace>/</robotNamespace>
+        </plugin>
+    </gazebo>
 </robot>

Commit message: added colour to links

File: urdf/diffDriveTest.urdf.xacro (robot description, xacro)
@@ -34,4 +34,7 @@
         <xacro:default_inertial mass="10"/>
     </link>
+    <gazebo reference="base_link">
+        <material>Gazebo/Orange</material>
+    </gazebo>
     <!-- wheels -->
     <xacro:macro name="wheels" params = "prefex reflect">
@@ -58,4 +61,7 @@
             <origin rpy="0 0 0" xyz="-${WheelPoss*2} ${reflect*WheelSep/2} -0.13"/>
         </joint>
+        <gazebo reference="${prefex}_back_wheel">
+            <material>Gazebo/Black</material>
+        </gazebo>
         <link name="${prefex}_back_M_wheel">
             <visual>
@@ -79,4 +85,7 @@
             <origin rpy="0 0 0" xyz="-${WheelPoss} ${reflect*WheelSep/2} -0.13"/>
         </joint>
+        <gazebo reference="${prefex}_back_M_wheel">
+            <material>Gazebo/Black</material>
+        </gazebo>
         <!-- front wheels -->
         <link name="${prefex}_front_M_wheel">
@@ -101,4 +110,7 @@
             <origin rpy="0 0 0" xyz="${WheelPoss} ${reflect*WheelSep/2} -0.13"/>
         </joint>
+        <gazebo reference="${prefex}_front_M_wheel">
+            <material>Gazebo/Black</material>
+        </gazebo>
         <link name="${prefex}_front_wheel">
             <visual>
@@ -122,4 +134,7 @@
             <origin rpy="0 0 0" xyz="${WheelPoss*2} ${reflect*WheelSep/2} -0.13"/>
         </joint>
+        <gazebo reference="${prefex}_front_wheel">
+            <material>Gazebo/Black</material>
+        </gazebo>
     </xacro:macro>
     <xacro:wheels prefex = "right" reflect = "-1"/>

Commit message: random commit

File: urdf/diffDriveTest.urdf.xacro (robot description, xacro)
@@ -59,5 +59,5 @@
             <parent link="base_link"/>
             <child link="${prefex}_back_wheel"/>
-            <origin rpy="0 0 0" xyz="-${WheelPoss*2} ${reflect*WheelSep/2} -0.13"/>
+            <origin rpy="0 0 0" xyz="-${WheelPoss*2} ${reflect*WheelSep/2} -0.15"/>
         </joint>
         <gazebo reference="${prefex}_back_wheel">
@@ -83,5 +83,5 @@
             <parent link="base_link"/>
             <child link="${prefex}_back_M_wheel"/>
-            <origin rpy="0 0 0" xyz="-${WheelPoss} ${reflect*WheelSep/2} -0.13"/>
+            <origin rpy="0 0 0" xyz="-${WheelPoss} ${reflect*WheelSep/2} -0.15"/>
         </joint>
         <gazebo reference="${prefex}_back_M_wheel">
@@ -108,5 +108,5 @@
             <parent link="base_link"/>
             <child link="${prefex}_front_M_wheel"/>
-            <origin rpy="0 0 0" xyz="${WheelPoss} ${reflect*WheelSep/2} -0.13"/>
+            <origin rpy="0 0 0" xyz="${WheelPoss} ${reflect*WheelSep/2} -0.15"/>
         </joint>
         <gazebo reference="${prefex}_front_M_wheel">
@@ -132,5 +132,5 @@
             <parent link="base_link"/>
             <child link="${prefex}_front_wheel"/>
-            <origin rpy="0 0 0" xyz="${WheelPoss*2} ${reflect*WheelSep/2} -0.13"/>
+            <origin rpy="0 0 0" xyz="${WheelPoss*2} ${reflect*WheelSep/2} -0.15"/>
         </joint>
         <gazebo reference="${prefex}_front_wheel">
@@ -163,5 +163,5 @@
             <wheelTorque>20</wheelTorque>
             <!-- Topic to receive geometry_msgs/Twist message commands, defaults to `cmd_vel` -->
-            <commandTopic>/diff_drive_controller/cmd_vel</commandTopic>
+            <commandTopic>diff_drive_controller/cmd_vel</commandTopic>
             <!-- Topic to publish nav_msgs/Odometry messages, defaults to `odom` -->
             <odometryTopic>odom</odometryTopic>
@@ -175,5 +175,5 @@
             <publishWheelTF>true</publishWheelTF>
             <!-- Set to true to publish transforms for the odometry, defaults to true -->
-            <publishOdom>true</publishOdom>
+            <publishOdomTF>true</publishOdomTF>
             <!-- Set to true to publish sensor_msgs/JointState on /joint_states for the wheel joints, defaults to false -->
             <publishWheelJointState>true</publishWheelJointState>

Commit message: random commit

File: urdf/diffDriveTest.urdf.xacro (robot description, xacro)
@@ -59,5 +59,5 @@
             <parent link="base_link"/>
             <child link="${prefex}_back_wheel"/>
-            <origin rpy="0 0 0" xyz="-${WheelPoss*2} ${reflect*WheelSep/2} -0.15"/>
+            <origin rpy="0 0 0" xyz="-${WheelPoss*2} ${reflect*WheelSep/2} -0.17"/>
         </joint>
         <gazebo reference="${prefex}_back_wheel">
@@ -83,5 +83,5 @@
             <parent link="base_link"/>
             <child link="${prefex}_back_M_wheel"/>
-            <origin rpy="0 0 0" xyz="-${WheelPoss} ${reflect*WheelSep/2} -0.15"/>
+            <origin rpy="0 0 0" xyz="-${WheelPoss} ${reflect*WheelSep/2} -0.17"/>
         </joint>
         <gazebo reference="${prefex}_back_M_wheel">
@@ -108,5 +108,5 @@
             <parent link="base_link"/>
             <child link="${prefex}_front_M_wheel"/>
-            <origin rpy="0 0 0" xyz="${WheelPoss} ${reflect*WheelSep/2} -0.15"/>
+            <origin rpy="0 0 0" xyz="${WheelPoss} ${reflect*WheelSep/2} -0.17"/>
         </joint>
         <gazebo reference="${prefex}_front_M_wheel">
@@ -132,5 +132,5 @@
             <parent link="base_link"/>
             <child link="${prefex}_front_wheel"/>
-            <origin rpy="0 0 0" xyz="${WheelPoss*2} ${reflect*WheelSep/2} -0.15"/>
+            <origin rpy="0 0 0" xyz="${WheelPoss*2} ${reflect*WheelSep/2} -0.17"/>
         </joint>
         <gazebo reference="${prefex}_front_wheel">

Commit message: random commit

File: urdf/diffDriveTest.urdf.xacro (robot description, xacro)
@@ -1,17 +1,9 @@
 <?xml version="1.0"?>
 <robot name="roscontrol" xmlns:xacro="http://ros.org/wiki/xacro">
-    <xacro:property name="WheelSep" value="0.26"/>
-    <xacro:property name="WheelRad" value="0.055"/>
-    <xacro:property name="WheelLen" value="0.1"/>
+    <xacro:property name="WheelSep" value="0.46"/>
+    <xacro:property name="WheelRad" value="0.06"/>
+    <xacro:property name="WheelLen" value="0.05"/>
     <xacro:property name="WheelPoss" value="0.15"/>
-    <material name="blue">
-        <color rgba="0 0 0.8 1"/>
-    </material>
-    <material name="black">
-        <color rgba="0 0 0 1"/>
-    </material>
-    <material name="white">
-        <color rgba="1 1 1 1"/>
-    </material>
+    <xacro:property name="WheelPossZ" value="-0.05"/>
     <xacro:macro name="default_inertial" params="mass">
         <inertial>
@@ -59,8 +51,16 @@
             <parent link="base_link"/>
             <child link="${prefex}_back_wheel"/>
-            <origin rpy="0 0 0" xyz="-${WheelPoss*2} ${reflect*WheelSep/2} -0.17"/>
+            <origin rpy="0 0 0" xyz="-${WheelPoss*2} ${reflect*WheelSep/2} ${WheelPossZ}"/>
         </joint>
         <gazebo reference="${prefex}_back_wheel">
             <material>Gazebo/Black</material>
+        </gazebo>
+        <gazebo reference="${prefex}_back_wheel">
+            <kp>1000000.0</kp>
+            <kd>1.0</kd>
+            <mu1>0.8</mu1>
+            <mu2>0.8</mu2>
+            <maxVel>0.0</maxVel>
+            <minDepth>0.001</minDepth>
         </gazebo>
         <link name="${prefex}_back_M_wheel">
@@ -83,8 +83,16 @@
             <parent link="base_link"/>
             <child link="${prefex}_back_M_wheel"/>
-            <origin rpy="0 0 0" xyz="-${WheelPoss} ${reflect*WheelSep/2} -0.17"/>
+            <origin rpy="0 0 0" xyz="-${WheelPoss} ${reflect*WheelSep/2} ${WheelPossZ}"/>
         </joint>
         <gazebo reference="${prefex}_back_M_wheel">
             <material>Gazebo/Black</material>
+        </gazebo>
+        <gazebo reference="${prefex}_back_M_wheel">
+            <kp>1000000.0</kp>
+            <kd>1.0</kd>
+            <mu1>0.8</mu1>
+            <mu2>0.8</mu2>
+            <maxVel>0.0</maxVel>
+            <minDepth>0.001</minDepth>
         </gazebo>
         <!-- front wheels -->
@@ -108,8 +116,16 @@
             <parent link="base_link"/>
             <child link="${prefex}_front_M_wheel"/>
-            <origin rpy="0 0 0" xyz="${WheelPoss} ${reflect*WheelSep/2} -0.17"/>
+            <origin rpy="0 0 0" xyz="${WheelPoss} ${reflect*WheelSep/2} ${WheelPossZ}"/>
         </joint>
         <gazebo reference="${prefex}_front_M_wheel">
             <material>Gazebo/Black</material>
+        </gazebo>
+        <gazebo reference="${prefex}_front_M_wheel">
+            <kp>1000000.0</kp>
+            <kd>1.0</kd>
+            <mu1>0.8</mu1>
+            <mu2>0.8</mu2>
+            <maxVel>0.0</maxVel>
+            <minDepth>0.001</minDepth>
         </gazebo>
         <link name="${prefex}_front_wheel">
@@ -132,8 +148,16 @@
             <parent link="base_link"/>
             <child link="${prefex}_front_wheel"/>
-            <origin rpy="0 0 0" xyz="${WheelPoss*2} ${reflect*WheelSep/2} -0.17"/>
+            <origin rpy="0 0 0" xyz="${WheelPoss*2} ${reflect*WheelSep/2} ${WheelPossZ}"/>
         </joint>
         <gazebo reference="${prefex}_front_wheel">
             <material>Gazebo/Black</material>
+        </gazebo>
+        <gazebo reference="${prefex}_front_wheel">
+            <kp>1000000.0</kp>
+            <kd>1.0</kd>
+            <mu1>0.8</mu1>
+            <mu2>0.8</mu2>
+            <maxVel>0.0</maxVel>
+            <minDepth>0.001</minDepth>
         </gazebo>
     </xacro:macro>
@@ -153,6 +177,6 @@
             <wheelSeparation>${WheelSep}</wheelSeparation>
             <wheelDiameter>${WheelRad*2}</wheelDiameter>
-            <wheelAcceleration>1.0</wheelAcceleration>
-            <wheelTorque>20</wheelTorque>
+            <wheelAcceleration>0.2</wheelAcceleration>
+            <wheelTorque>5</wheelTorque>
             <commandTopic>diff_drive_controller/cmd_vel</commandTopic>
             <odometryTopic>odom</odometryTopic>
