Commit message: random commit

File: urdf/diffDriveTest.xacro (robot description, xacro)
@@ -2,5 +2,5 @@
 <robot name="roscontrol" xmlns:xacro="http://ros.org/wiki/xacro">
     <xacro:property name="WheelSep" value="0.46"/>
-    <xacro:property name="WheelRad" value="0.06"/>
+    <xacro:property name="WheelRad" value="0.1"/>
     <xacro:property name="WheelLen" value="0.05"/>
     <xacro:property name="WheelPoss" value="0.15"/>
@@ -13,9 +13,9 @@
     </xacro:macro>
     <link name="base_link">
+        <pose>0 0 0.1 0 0 0</pose>
         <visual>
             <geometry>
                 <box size="0.8 0.4 0.2"/>
             </geometry>
-            <material name="blue"/>
         </visual>
         <collision>
@@ -24,8 +24,8 @@
             </geometry>
         </collision>
-        <xacro:default_inertial mass="10"/>
+        <xacro:default_inertial mass="15"/>
     </link>
     <gazebo reference="base_link">
-        <material>Gazebo/Orange</material>
+        <material>Gazebo/Blue</material>
     </gazebo>
     <!-- wheels -->
@@ -34,16 +34,16 @@
         <link name="${prefex}_back_wheel">
             <visual>
-                <origin rpy="1.57075 0 0" xyz="0 0 0"/>
+                <origin xyz="0 0 0" rpy="0 1.5707 1.5707"/>
                 <geometry>
                     <cylinder length="${WheelLen}" radius="${WheelRad}"/>
                 </geometry>
-                <material name="black"/>
             </visual>
             <collision>
+                <origin xyz="0 0 0" rpy="0 1.5707 1.5707"/>
                 <geometry>
                     <cylinder length="${WheelLen}" radius="${WheelRad}"/>
                 </geometry>
             </collision>
-            <xacro:default_inertial mass="1"/>
+            <xacro:default_inertial mass="5"/>
         </link>
         <joint name="${prefex}_back_wheel_joint" type="continuous">
@@ -52,95 +52,52 @@
             <child link="${prefex}_back_wheel"/>
             <origin rpy="0 0 0" xyz="-${WheelPoss*2} ${reflect*WheelSep/2} ${WheelPossZ}"/>
+            <limit effort="10000" velocity="1000"/>
+            <dynamics damping="1.0" friction="1.0"/>
         </joint>
         <gazebo reference="${prefex}_back_wheel">
             <material>Gazebo/Black</material>
         </gazebo>
-        <gazebo reference="${prefex}_back_wheel">
-            <kp>1000000.0</kp>
-            <kd>1.0</kd>
-            <mu1>0.8</mu1>
-            <mu2>0.8</mu2>
-            <maxVel>0.0</maxVel>
-            <minDepth>0.001</minDepth>
-        </gazebo>
-        <link name="${prefex}_back_M_wheel">
+        <!-- middle wheels -->
+        <link name="${prefex}_middle_wheel">
             <visual>
-                <origin rpy="1.57075 0 0" xyz="0 0 0"/>
+                <origin xyz="0 0 0" rpy="0 1.5707 1.5707"/>
                 <geometry>
                     <cylinder length="${WheelLen}" radius="${WheelRad}"/>
                 </geometry>
-                <material name="black"/>
             </visual>
             <collision>
+                <origin xyz="0 0 0" rpy="0 1.5707 1.5707"/>
                 <geometry>
                     <cylinder length="${WheelLen}" radius="${WheelRad}"/>
                 </geometry>
             </collision>
-            <xacro:default_inertial mass="1"/>
+            <xacro:default_inertial mass="5"/>
         </link>
-        <joint name="${prefex}_back_M_wheel_joint" type="continuous">
+        <joint name="${prefex}_middle_wheel_joint" type="continuous">
             <axis xyz="0 1 0" rpy="0 0 0" />
             <parent link="base_link"/>
-            <child link="${prefex}_back_M_wheel"/>
-            <origin rpy="0 0 0" xyz="-${WheelPoss} ${reflect*WheelSep/2} ${WheelPossZ}"/>
+            <child link="${prefex}_middle_wheel"/>
+            <origin rpy="0 0 0" xyz="0 ${reflect*WheelSep/2} ${WheelPossZ}"/>
+            <limit effort="10000" velocity="1000"/>
+            <dynamics damping="1.0" friction="1.0"/>
         </joint>
-        <gazebo reference="${prefex}_back_M_wheel">
+        <gazebo reference="${prefex}_middle_wheel">
             <material>Gazebo/Black</material>
         </gazebo>
-        <gazebo reference="${prefex}_back_M_wheel">
-            <kp>1000000.0</kp>
-            <kd>1.0</kd>
-            <mu1>0.8</mu1>
-            <mu2>0.8</mu2>
-            <maxVel>0.0</maxVel>
-            <minDepth>0.001</minDepth>
-        </gazebo>
         <!-- front wheels -->
-        <link name="${prefex}_front_M_wheel">
+        <link name="${prefex}_front_wheel">
             <visual>
-                <origin rpy="1.57075 0 0" xyz="0 0 0"/>
+                <origin xyz="0 0 0" rpy="0 1.5707 1.5707"/>
                 <geometry>
                     <cylinder length="${WheelLen}" radius="${WheelRad}"/>
                 </geometry>
-                <material name="black"/>
             </visual>
             <collision>
+                <origin xyz="0 0 0" rpy="0 1.5707 1.5707"/>
                 <geometry>
                     <cylinder length="${WheelLen}" radius="${WheelRad}"/>
                 </geometry>
             </collision>
-            <xacro:default_inertial mass="1"/>
-        </link>
-        <joint name="${prefex}_front_M_wheel_joint" type="continuous">
-            <axis xyz="0 1 0" rpy="0 0 0" />
-            <parent link="base_link"/>
-            <child link="${prefex}_front_M_wheel"/>
-            <origin rpy="0 0 0" xyz="${WheelPoss} ${reflect*WheelSep/2} ${WheelPossZ}"/>
-        </joint>
-        <gazebo reference="${prefex}_front_M_wheel">
-            <material>Gazebo/Black</material>
-        </gazebo>
-        <gazebo reference="${prefex}_front_M_wheel">
-            <kp>1000000.0</kp>
-            <kd>1.0</kd>
-            <mu1>0.8</mu1>
-            <mu2>0.8</mu2>
-            <maxVel>0.0</maxVel>
-            <minDepth>0.001</minDepth>
-        </gazebo>
-        <link name="${prefex}_front_wheel">
-            <visual>
-                <origin rpy="1.57075 0 0" xyz="0 0 0"/>
-                <geometry>
-                    <cylinder length="${WheelLen}" radius="${WheelRad}"/>
-                </geometry>
-                <material name="black"/>
-            </visual>
-            <collision>
-                <geometry>
-                    <cylinder length="${WheelLen}" radius="${WheelRad}"/>
-                </geometry>
-            </collision>
-            <xacro:default_inertial mass="1"/>
+            <xacro:default_inertial mass="5"/>
         </link>
         <joint name="${prefex}_front_wheel_joint" type="continuous">
@@ -149,15 +106,9 @@
             <child link="${prefex}_front_wheel"/>
             <origin rpy="0 0 0" xyz="${WheelPoss*2} ${reflect*WheelSep/2} ${WheelPossZ}"/>
+            <limit effort="10000" velocity="1000"/>
+            <dynamics damping="1.0" friction="1.0"/>
         </joint>
         <gazebo reference="${prefex}_front_wheel">
             <material>Gazebo/Black</material>
-        </gazebo>
-        <gazebo reference="${prefex}_front_wheel">
-            <kp>1000000.0</kp>
-            <kd>1.0</kd>
-            <mu1>0.8</mu1>
-            <mu2>0.8</mu2>
-            <maxVel>0.0</maxVel>
-            <minDepth>0.001</minDepth>
         </gazebo>
     </xacro:macro>
@@ -173,6 +124,6 @@
         <plugin name="differential_drive_controller" filename="libgazebo_ros_diff_drive_multiwheel.so">
             <updateRate>50</updateRate>
-            <leftJoints>left_back_wheel_joint left_back_M_wheel_joint left_front_M_wheel_joint left_front_wheel_joint</leftJoints>
-            <rightJoints>right_back_wheel_joint right_back_M_wheel_joint right_front_M_wheel_joint right_front_wheel_joint</rightJoints>
+            <leftJoints>left_back_wheel_joint left_middle_wheel_joint left_front_wheel_joint</leftJoints>
+            <rightJoints>right_back_wheel_joint right_middle_wheel_joint right_front_wheel_joint</rightJoints>
             <wheelSeparation>${WheelSep}</wheelSeparation>
             <wheelDiameter>${WheelRad*2}</wheelDiameter>

File: urdf/twoWheelsRobot.xacro (robot description, xacro)
@@ -1,12 +1,5 @@
 <?xml version='1.0'?>
-<robot name="my_robot" xmlns:xacro="http://www.ros.org/wiki/xacro">
-  <xacro:include filename="$(find gazebo_ros_diff_drive_multiwheel)/urdf/my_robot.gazebo" />
-  <link name="robot_footprint"></link>
-  <joint name="robot_footprint_joint" type="fixed">
-    <origin xyz="0 0 0" rpy="0 0 0" />
-    <parent link="robot_footprint"/>
-    <child link="chassis" />
-  </joint>
-  <link name='chassis'>
+<robot name="twoWheelsRobot" xmlns:xacro="http://www.ros.org/wiki/xacro">
+  <link name='base_link'>
     <pose>0 0 0.1 0 0 0</pose>
     <inertial>
@@ -25,5 +18,5 @@
       </geometry>
     </collision>
-    <visual name='chassis_visual'>
+    <visual name='base_link_visual'>
       <origin xyz="0 0 0" rpy=" 0 0 0"/>
       <geometry>
@@ -59,5 +52,5 @@
     <origin xyz="0 0.15 0" rpy="0 0 0"/>
     <child link="left_wheel"/>
-    <parent link="chassis"/>
+    <parent link="base_link"/>
     <axis xyz="0 1 0" rpy="0 0 0"/>
     <limit effort="10000" velocity="1000"/>
@@ -90,5 +83,5 @@
     <origin xyz="0 -0.15 0" rpy="0 0 0"/>
     <child link="right_wheel"/>
-    <parent link="chassis"/>
+    <parent link="base_link"/>
     <axis xyz="0 1 0" rpy="0 0 0"/>
     <limit effort="10000" velocity="1000"/>
@@ -119,14 +112,31 @@
   </link>
   <gazebo reference="left_wheel">
-    <material>Gazebo/Green</material>
+    <material>Gazebo/Black</material>
   </gazebo>
   <gazebo reference="right_wheel">
-    <material>Gazebo/Green</material>
+    <material>Gazebo/Black</material>
   </gazebo>
-  <gazebo reference="camera">
-    <material>Gazebo/Red</material>
-  </gazebo>
-  <gazebo reference="chassis">
+  <gazebo reference="base_link">
     <material>Gazebo/Blue</material>
   </gazebo>
+  <gazebo>
+    <plugin name="differential_drive_controller" filename="libgazebo_ros_diff_drive_multiwheel.so">
+      <updateRate>50</updateRate>
+      <leftJoints>left_wheel_hinge</leftJoints>
+      <rightJoints>right_wheel_hinge</rightJoints>
+      <wheelSeparation>0.4</wheelSeparation>
+      <wheelDiameter>0.2</wheelDiameter>
+      <wheelAcceleration>0.2</wheelAcceleration>
+      <wheelTorque>5</wheelTorque>
+      <commandTopic>diff_drive_controller/cmd_vel</commandTopic>
+      <odometryTopic>odom</odometryTopic>
+      <odometryFrame>odom</odometryFrame>
+      <robotBaseFrame>base_link</robotBaseFrame>
+      <odometrySource>1</odometrySource>
+      <publishWheelTF>true</publishWheelTF>
+      <publishOdomTF>true</publishOdomTF>
+      <publishWheelJointState>true</publishWheelJointState>
+      <legacyMode>false</legacyMode>
+    </plugin>
+  </gazebo>
 </robot>

Commit message: random commit

File: urdf/diffDriveTest.xacro (robot description, xacro)
@@ -58,4 +58,25 @@
             <material>Gazebo/Black</material>
         </gazebo>
+        <link name="${prefex}_column_back">
+            <visual>
+                <geometry>
+                    <box size="0.01 0.04 0.02"/>
+                </geometry>
+            </visual>
+            <collision>
+                <geometry>
+                    <box size="0.01 0.04 0.02"/>
+                </geometry>
+            </collision>
+            <xacro:default_inertial mass="0.01"/>
+        </link>
+        <joint name="${prefex}_back_wheel_coll_joint" type="fixed">
+            <child link="${prefex}_column_back"/>
+            <parent link="${prefex}_back_wheel"/>
+            <origin rpy="0 0 0" xyz="0.06 ${reflect*0.01} 0"/>
+        </joint>
+        <gazebo reference="${prefex}_column_back">
+            <material>Gazebo/White</material>
+        </gazebo>
         <!-- middle wheels -->
         <link name="${prefex}_middle_wheel">
@@ -85,4 +106,25 @@
             <material>Gazebo/Black</material>
         </gazebo>
+        <link name="${prefex}_column_middle">
+            <visual>
+                <geometry>
+                    <box size="0.01 0.04 0.02"/>
+                </geometry>
+            </visual>
+            <collision>
+                <geometry>
+                    <box size="0.01 0.04 0.02"/>
+                </geometry>
+            </collision>
+            <xacro:default_inertial mass="0.01"/>
+        </link>
+        <joint name="${prefex}_middle_wheel_coll_joint" type="fixed">
+            <child link="${prefex}_column_middle"/>
+            <parent link="${prefex}_middle_wheel"/>
+            <origin rpy="0 0 0" xyz="0.06 ${reflect*0.01} 0"/>
+        </joint>
+        <gazebo reference="${prefex}_column_middle">
+            <material>Gazebo/White</material>
+        </gazebo>
         <!-- front wheels -->
         <link name="${prefex}_front_wheel">
@@ -111,4 +153,25 @@
         <gazebo reference="${prefex}_front_wheel">
             <material>Gazebo/Black</material>
+        </gazebo>
+        <link name="${prefex}_column_front">
+            <visual>
+                <geometry>
+                    <box size="0.01 0.04 0.02"/>
+                </geometry>
+            </visual>
+            <collision>
+                <geometry>
+                    <box size="0.01 0.04 0.02"/>
+                </geometry>
+            </collision>
+            <xacro:default_inertial mass="0.01"/>
+        </link>
+        <joint name="${prefex}_front_wheel_coll_joint" type="fixed">
+            <child link="${prefex}_column_front"/>
+            <parent link="${prefex}_front_wheel"/>
+            <origin rpy="0 0 0" xyz="0.06 ${reflect*0.01} 0"/>
+        </joint>
+        <gazebo reference="${prefex}_column_front">
+            <material>Gazebo/White</material>
         </gazebo>
     </xacro:macro>
